Commit message: Update URDF: replaced 3D LiDAR with 2D LiDAR sensor

File: urdf/jetbot_csi.gazebo.xacro (robot description, xacro)
@@ -1,8 +1,8 @@
 <?xml version="1.0"?>
 <robot name="turtlebot3_burger_sim" xmlns:xacro="http://ros.org/wiki/xacro">
-  <xacro:arg name="laser_visual" default="false"/>
+  <xacro:arg name="laser_visual" default="true"/>
   <xacro:arg name="imu_visual"   default="false"/>
   <xacro:property name="M_PI" value="3.14159265359"/>
-  <xacro:property name="use_Rplidar" default="false"/>
+  <xacro:property name="use_Rplidar" default="true"/>
   <gazebo reference="base_link">
     <material>Gazebo/Green</material>
@@ -142,5 +142,5 @@
       </plugin>
     </gazebo>
-      <!-- <gazebo reference="base_scan">
+      <gazebo reference="base_scan">
         <material>Gazebo/FlatBlack</material>
         <sensor type="ray" name="lds_lfcd_sensor">
@@ -173,6 +173,6 @@
           </plugin>
         </sensor>
-      </gazebo> -->
-    <gazebo reference="base_scan">
+      </gazebo>
+    <!-- <gazebo reference="base_scan">
       <material>Gazebo/FlatBlack</material>
       <sensor type="ray" name="velodyne-VLP16">
@@ -215,4 +215,4 @@
         </plugin>
       </sensor>
-    </gazebo>
+    </gazebo> -->
 </robot>

File: urdf/jetbot_real.gazebo.xacro (robot description, xacro)
@@ -1,5 +1,5 @@
 <?xml version="1.0"?>
 <robot name="turtlebot3_burger_sim" xmlns:xacro="http://ros.org/wiki/xacro">
-  <xacro:arg name="laser_visual" default="false" />
+  <xacro:arg name="laser_visual" default="true" />
   <xacro:arg name="imu_visual"   default="false"/>
   <gazebo reference="base_link">
@@ -46,5 +46,5 @@
   </gazebo>
   <!--base_scan-->
- <!-- <gazebo reference="base_scan">
+  <gazebo reference="base_scan">
     <sensor type="camera" name="camera1">
       <update_rate>30.0</update_rate>
@@ -80,5 +80,5 @@
       </plugin>
     </sensor>
-  </gazebo> -->
+  </gazebo>
   <gazebo reference="wheel_left_link">
     <mu1>0.1</mu1>
@@ -176,5 +176,5 @@
     </plugin>
   </gazebo>
-  <!-- <gazebo reference="base_scan">
+  <gazebo reference="base_scan">
     <material>Gazebo/FlatBlack</material>
     <sensor type="ray" name="lds_lfcd_sensor">
@@ -207,6 +207,6 @@
       </plugin>
     </sensor>
-  </gazebo> -->
-      <gazebo reference="base_scan">
+  </gazebo>
+      <!-- <gazebo reference="base_scan">
       <material>Gazebo/FlatBlack</material>
       <sensor type="ray" name="velodyne-VLP16">
@@ -249,4 +249,4 @@
         </plugin>
       </sensor>
-    </gazebo>
+    </gazebo> -->
 </robot>
