Commit message: Modified URDF files: changed STL file directory

File: urdf/jetbot_csi.urdf (robot description, URDF)
Before this commit: robot Jetbot, 21 links, 20 joints
Links:
- link antenna_link: geometry collision mesh filename=package://jetbot_world/meshes/other_parts/antenna_link.STL; visual mesh filename=package://jetbot_world/meshes/other_parts/antenna_link.STL
- link base_link: geometry collision mesh filename=package://jetbot_world/meshes/other_parts/base_link.STL; visual mesh filename=package://jetbot_world/meshes/other_parts/base_link.STL
- link base_scan: geometry collision mesh filename=package://jetbot_world/meshes/other_parts/base_scan.STL; visual mesh filename=package://jetbot_world/meshes/other_parts/base_scan.STL
- link bolt1_link: geometry collision mesh filename=package://jetbot_world/meshes/other_parts/bolt1_link.STL; visual mesh filename=package://jetbot_world/meshes/other_parts/bolt1_link.STL
- link bolt2_link: geometry collision mesh filename=package://jetbot_world/meshes/other_parts/bolt2_link.STL; visual mesh filename=package://jetbot_world/meshes/other_parts/bolt2_link.STL
- link camera_link: geometry collision mesh filename=package://jetbot_world/meshes/csi/camera_link.STL; visual mesh filename=package://jetbot_world/meshes/csi/camera_link.STL
- link camera_mount_link: geometry collision mesh filename=package://jetbot_world/meshes/csi/camera_mount_link.STL; visual mesh filename=package://jetbot_world/meshes/csi/camera_mount_link.STL
- link caster_back_link: geometry collision mesh filename=package://jetbot_world/meshes/other_parts/caster_back_link.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; visual mesh filename=package://jetbot_world/meshes/other_parts/caster_back_link.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
- link caster_front_link: geometry collision mesh filename=package://jetbot_world/meshes/other_parts/caster_front_link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; visual mesh filename=package://jetbot_world/meshes/other_parts/caster_front_link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
- link imu_link: geometry collision mesh filename=package://jetbot_world/meshes/other_parts/imu_link.STL; visual mesh filename=package://jetbot_world/meshes/other_parts/imu_link.STL
- link left_motor_link: geometry collision mesh filename=package://jetbot_world/meshes/other_parts/left_motor_link.S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; visual mesh filename=package://jetbot_world/meshes/other_parts/left_motor_link.S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
- link nano_link: geometry collision mesh filename=package://jetbot_world/meshes/other_parts/nano_link.STL; visual mesh filename=package://jetbot_world/meshes/other_parts/nano_link.STL
- link right_motor_link: geometry collision mesh filename=package://jetbot_world/meshes/other_parts/right_motor_link.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; visual mesh filename=package://jetbot_world/meshes/other_parts/right_motor_link.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
- link upper_plate_link: geometry collision mesh filename=package://jetbot_world/meshes/other_parts/upper_plate_link.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; visual mesh filename=package://jetbot_world/meshes/other_parts/upper_plate_link.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
- link wheel_left_link: geometry collision mesh filename=package://jetbot_world/meshes/wheels/wheel_left_link.STL; visual mesh filename=package://jetbot_world/meshes/wheels/wheel_left_link.STL
- link wheel_left_rim: geometry collision mesh filename=package://jetbot_world/meshes/wheels/wheel_left_rim.STL; visual mesh filename=package://jetbot_world/meshes/wheels/wheel_left_rim.STL
- link wheel_left_tire: geometry collision mesh filename=package://jetbot_world/meshes/wheels/wheel_left_tire.STL; visual mesh filename=package://jetbot_world/meshes/wheels/wheel_left_tire.STL
- link wheel_right_link: geometry collision mesh filename=package://jetbot_world/meshes/wheels/wheel_right_link.STL; visual mesh filename=package://jetbot_world/meshes/wheels/wheel_right_link.STL
- link wheel_right_rim: geometry collision mesh filename=package://jetbot_world/meshes/wheels/wheel_right_rim.STL; visual mesh filename=package://jetbot_world/meshes/wheels/wheel_right_rim.STL
- link wheel_right_tire: geometry collision mesh filename=package://jetbot_world/meshes/wheels/wheel_right_tire.STL; visual mesh filename=package://jetbot_world/meshes/wheels/wheel_right_tire.STL

File: urdf/jetbot_csi.urdf.xacro (robot description, xacro)
@@ -25,5 +25,5 @@
       <origin rpy="0 0 0" xyz="0 0 0"/>
       <geometry>
-        <mesh filename="package://jetbot_model/meshes/other_parts/base_link.STL"/>
+        <mesh filename="package://jetbot_world/meshes/other_parts/base_link.STL"/>
       </geometry>
       <material name="">
@@ -34,5 +34,5 @@
       <origin rpy="0 0 0" xyz="0 0 0"/>
       <geometry>
-        <mesh filename="package://jetbot_model/meshes/other_parts/base_link.STL"/>
+        <mesh filename="package://jetbot_world/meshes/other_parts/base_link.STL"/>
       </geometry>
     </collision>
@@ -47,5 +47,5 @@
       <origin rpy="0 0 0" xyz="0 0 0"/>
       <geometry>
-        <mesh filename="package://jetbot_model/meshes/wheels/wheel_right_link.STL"/>
+        <mesh filename="package://jetbot_world/meshes/wheels/wheel_right_link.STL"/>
       </geometry>
       <material name="">
@@ -56,5 +56,5 @@
       <origin rpy="0 0 0" xyz="0 0 0"/>
       <geometry>
-        <mesh filename="package://jetbot_model/meshes/wheels/wheel_right_link.STL"/>
+        <mesh filename="package://jetbot_world/meshes/wheels/wheel_right_link.STL"/>
       </geometry>
     </collision>
@@ -76,5 +76,5 @@
       <origin rpy="0 0 0" xyz="0 0 0"/>
       <geometry>
-        <mesh filename="package://jetbot_model/meshes/wheels/wheel_right_rim.STL"/>
+        <mesh filename="package://jetbot_world/meshes/wheels/wheel_right_rim.STL"/>
       </geometry>
       <material name="">
@@ -85,5 +85,5 @@
       <origin rpy="0 0 0" xyz="0 0 0"/>
       <geometry>
-        <mesh filename="package://jetbot_model/meshes/wheels/wheel_right_rim.STL"/>
+        <mesh filename="package://jetbot_world/meshes/wheels/wheel_right_rim.STL"/>
       </geometry>
     </collision>
@@ -104,5 +104,5 @@
       <origin rpy="0 0 0" xyz="0 0 0"/>
       <geometry>
-        <mesh filename="package://jetbot_model/meshes/wheels/wheel_right_tire.STL"/>
+        <mesh filename="package://jetbot_world/meshes/wheels/wheel_right_tire.STL"/>
       </geometry>
       <material name="">
@@ -113,5 +113,5 @@
       <origin rpy="0 0 0" xyz="0 0 0"/>
       <geometry>
-        <mesh filename="package://jetbot_model/meshes/wheels/wheel_right_tire.STL"/>
+        <mesh filename="package://jetbot_world/meshes/wheels/wheel_right_tire.STL"/>
       </geometry>
     </collision>
@@ -132,5 +132,5 @@
       <origin rpy="0 0 0" xyz="0 0 0"/>
       <geometry>
-        <mesh filename="package://jetbot_model/meshes/wheels/wheel_left_link.STL"/>
+        <mesh filename="package://jetbot_world/meshes/wheels/wheel_left_link.STL"/>
       </geometry>
       <material name="">
@@ -141,5 +141,5 @@
       <origin rpy="0 0 0" xyz="0 0 0"/>
       <geometry>
-        <mesh filename="package://jetbot_model/meshes/wheels/wheel_left_link.STL"/>
+        <mesh filename="package://jetbot_world/meshes/wheels/wheel_left_link.STL"/>
       </geometry>
     </collision>
@@ -161,5 +161,5 @@
       <origin rpy="0 0 0" xyz="0 0 0"/>
       <geometry>
-        <mesh filename="package://jetbot_model/meshes/wheels/wheel_left_rim.STL"/>
+        <mesh filename="package://jetbot_world/meshes/wheels/wheel_left_rim.STL"/>
       </geometry>
       <material name="">
@@ -170,5 +170,5 @@
       <origin rpy="0 0 0" xyz="0 0 0"/>
       <geometry>
-        <mesh filename="package://jetbot_model/meshes/wheels/wheel_left_rim.STL"/>
+        <mesh filename="package://jetbot_world/meshes/wheels/wheel_left_rim.STL"/>
       </geometry>
     </collision>
@@ -189,5 +189,5 @@
       <origin rpy="0 0 0" xyz="0 0 0"/>
       <geometry>
-        <mesh filename="package://jetbot_model/meshes/wheels/wheel_left_tire.STL"/>
+        <mesh filename="package://jetbot_world/meshes/wheels/wheel_left_tire.STL"/>
       </geometry>
       <material name="">
@@ -198,5 +198,5 @@
       <origin rpy="0 0 0" xyz="0 0 0"/>
       <geometry>
-        <mesh filename="package://jetbot_model/meshes/wheels/wheel_left_tire.STL"/>
+        <mesh filename="package://jetbot_world/meshes/wheels/wheel_left_tire.STL"/>
       </geometry>
     </collision>
@@ -217,5 +217,5 @@
       <origin rpy="0 0 0" xyz="0 0 0"/>
       <geometry>
-        <mesh filename="package://jetbot_model/meshes/csi/camera_mount_link.STL"/>
+        <mesh filename="package://jetbot_world/meshes/csi/camera_mount_link.STL"/>
       </geometry>
       <material name="">
@@ -226,5 +226,5 @@
       <origin rpy="0 0 0" xyz="0 0 0"/>
       <geometry>
-        <mesh filename="package://jetbot_model/meshes/csi/camera_mount_link.STL"/>
+        <mesh filename="package://jetbot_world/meshes/csi/camera_mount_link.STL"/>
       </geometry>
     </collision>
@@ -245,5 +245,5 @@
       <origin rpy="0 0 0" xyz="0 0 0"/>
       <geometry>
-        <mesh filename="package://jetbot_model/meshes/csi/camera_link.STL"/>
+        <mesh filename="package://jetbot_world/meshes/csi/camera_link.STL"/>
       </geometry>
       <material name="">
@@ -254,5 +254,5 @@
       <origin rpy="0 0 0" xyz="0 0 0"/>
       <geometry>
-        <mesh filename="package://jetbot_model/meshes/csi/camera_link.STL"/>
+        <mesh filename="package://jetbot_world/meshes/csi/camera_link.STL"/>
       </geometry>
     </collision>
@@ -273,5 +273,5 @@
       <origin rpy="0 0 0" xyz="0 0 0"/>
       <geometry>
-        <mesh filename="package://jetbot_model/meshes/other_parts/caster_back_link.STL"/>
+        <mesh filename="package://jetbot_world/meshes/other_parts/caster_back_link.STL"/>
       </geometry>
       <material name="">
@@ -282,5 +282,5 @@
       <origin rpy="0 0 0" xyz="0 0 0"/>
       <geometry>
-        <mesh filename="package://jetbot_model/meshes/other_parts/caster_back_link.STL"/>
+        <mesh filename="package://jetbot_world/meshes/other_parts/caster_back_link.STL"/>
       </geometry>
     </collision>
@@ -301,5 +301,5 @@
       <origin rpy="0 0 0" xyz="0 0 0"/>
       <geometry>
-        <mesh filename="package://jetbot_model/meshes/other_parts/caster_front_link.STL"/>
+        <mesh filename="package://jetbot_world/meshes/other_parts/caster_front_link.STL"/>
       </geometry>
       <material name="">
@@ -310,5 +310,5 @@
       <origin rpy="0 0 0" xyz="0 0 0"/>
       <geometry>
-        <mesh filename="package://jetbot_model/meshes/other_parts/caster_front_link.STL"/>
+        <mesh filename="package://jetbot_world/meshes/other_parts/caster_front_link.STL"/>
       </geometry>
     </collision>
@@ -329,5 +329,5 @@
       <origin rpy="0 0 0" xyz="0 0 0"/>
       <geometry>
-        <mesh filename="package://jetbot_model/meshes/other_parts/imu_link.STL"/>
+        <mesh filename="package://jetbot_world/meshes/other_parts/imu_link.STL"/>
       </geometry>
       <material name="">
@@ -338,5 +338,5 @@
       <origin rpy="0 0 0" xyz="0 0 0"/>
       <geometry>
-        <mesh filename="package://jetbot_model/meshes/other_parts/imu_link.STL"/>
+        <mesh filename="package://jetbot_world/meshes/other_parts/imu_link.STL"/>
       </geometry>
     </collision>
@@ -357,5 +357,5 @@
       <origin rpy="0 0 0" xyz="0 0 0"/>
       <geometry>
-        <mesh filename="package://jetbot_model/meshes/other_parts/base_scan.STL"/>
+        <mesh filename="package://jetbot_world/meshes/other_parts/base_scan.STL"/>
       </geometry>
       <material name="">
@@ -366,5 +366,5 @@
       <origin rpy="0 0 0" xyz="0 0 0"/>
       <geometry>
-        <mesh filename="package://jetbot_model/meshes/other_parts/base_scan.STL"/>
+        <mesh filename="package://jetbot_world/meshes/other_parts/base_scan.STL"/>
       </geometry>
     </collision>
@@ -385,5 +385,5 @@
       <origin rpy="0 0 0" xyz="0 0 0"/>
       <geometry>
-        <mesh filename="package://jetbot_model/meshes/other_parts/left_motor_link.STL"/>
+        <mesh filename="package://jetbot_world/meshes/other_parts/left_motor_link.STL"/>
       </geometry>
       <material name="">
@@ -394,5 +394,5 @@
       <origin rpy="0 0 0" xyz="0 0 0"/>
       <geometry>
-        <mesh filename="package://jetbot_model/meshes/other_parts/left_motor_link.STL"/>
+        <mesh filename="package://jetbot_world/meshes/other_parts/left_motor_link.STL"/>
       </geometry>
     </collision>
@@ -413,5 +413,5 @@
       <origin rpy="0 0 0" xyz="0 0 0"/>
       <geometry>
-        <mesh filename="package://jetbot_model/meshes/other_parts/right_motor_link.STL"/>
+        <mesh filename="package://jetbot_world/meshes/other_parts/right_motor_link.STL"/>
       </geometry>
       <material name="">
@@ -422,5 +422,5 @@
       <origin rpy="0 0 0" xyz="0 0 0"/>
       <geometry>
-        <mesh filename="package://jetbot_model/meshes/other_parts/right_motor_link.STL"/>
+        <mesh filename="package://jetbot_world/meshes/other_parts/right_motor_link.STL"/>
       </geometry>
     </collision>
@@ -441,5 +441,5 @@
       <origin rpy="0 0 0" xyz="0 0 0"/>
       <geometry>
-        <mesh filename="package://jetbot_model/meshes/other_parts/upper_plate_link.STL"/>
+        <mesh filename="package://jetbot_world/meshes/other_parts/upper_plate_link.STL"/>
       </geometry>
       <material name="">
@@ -450,5 +450,5 @@
       <origin rpy="0 0 0" xyz="0 0 0"/>
       <geometry>
-        <mesh filename="package://jetbot_model/meshes/other_parts/upper_plate_link.STL"/>
+        <mesh filename="package://jetbot_world/meshes/other_parts/upper_plate_link.STL"/>
       </geometry>
     </collision>
@@ -469,5 +469,5 @@
       <origin rpy="0 0 0" xyz="0 0 0"/>
       <geometry>
-        <mesh filename="package://jetbot_model/meshes/other_parts/antenna_link.STL"/>
+        <mesh filename="package://jetbot_world/meshes/other_parts/antenna_link.STL"/>
       </geometry>
       <material name="">
@@ -478,5 +478,5 @@
       <origin rpy="0 0 0" xyz="0 0 0"/>
       <geometry>
-        <mesh filename="package://jetbot_model/meshes/other_parts/antenna_link.STL"/>
+        <mesh filename="package://jetbot_world/meshes/other_parts/antenna_link.STL"/>
       </geometry>
     </collision>
@@ -497,5 +497,5 @@
       <origin rpy="0 0 0" xyz="0 0 0"/>
       <geometry>
-        <mesh filename="package://jetbot_model/meshes/other_parts/bolt1_link.STL"/>
+        <mesh filename="package://jetbot_world/meshes/other_parts/bolt1_link.STL"/>
       </geometry>
       <material name="">
@@ -506,5 +506,5 @@
       <origin rpy="0 0 0" xyz="0 0 0"/>
       <geometry>
-        <mesh filename="package://jetbot_model/meshes/other_parts/bolt1_link.STL"/>
+        <mesh filename="package://jetbot_world/meshes/other_parts/bolt1_link.STL"/>
       </geometry>
     </collision>
@@ -525,5 +525,5 @@
       <origin rpy="0 0 0" xyz="0 0 0"/>
       <geometry>
-        <mesh filename="package://jetbot_model/meshes/other_parts/bolt2_link.STL"/>
+        <mesh filename="package://jetbot_world/meshes/other_parts/bolt2_link.STL"/>
       </geometry>
       <material name="">
@@ -534,5 +534,5 @@
       <origin rpy="0 0 0" xyz="0 0 0"/>
       <geometry>
-        <mesh filename="package://jetbot_model/meshes/other_parts/bolt2_link.STL"/>
+        <mesh filename="package://jetbot_world/meshes/other_parts/bolt2_link.STL"/>
       </geometry>
     </collision>
@@ -553,5 +553,5 @@
       <origin rpy="0 0 0" xyz="0 0 0"/>
       <geometry>
-        <mesh filename="package://jetbot_model/meshes/other_parts/nano_link.STL"/>
+        <mesh filename="package://jetbot_world/meshes/other_parts/nano_link.STL"/>
       </geometry>
       <material name="">
@@ -562,5 +562,5 @@
       <origin rpy="0 0 0" xyz="0 0 0"/>
       <geometry>
-        <mesh filename="package://jetbot_model/meshes/other_parts/nano_link.STL"/>
+        <mesh filename="package://jetbot_world/meshes/other_parts/nano_link.STL"/>
       </geometry>
     </collision>
